File: hardware/Schaltplan/Nanocopter_V2.brd (EAGLE design)
At the start: 100 x 100 mm, 86 parts, among them M1+ TPTP15SQ, M1- TPTP15SQ, M2+ TPTP15SQ, M2- TPTP15SQ, M3+ TPTP15SQ, M3- TPTP15SQ, M4+ TPTP15SQ, M4- TPTP15SQ, T1 IRLML2502, T2 IRLML2502, T3 IRLML2502, T4 IRLML2502, U1 MAX682, U2 PRTR5V0U2X, U3 LM3480-3.3, X1 USBSMD

Commit message: Arbeit an Schaltplan V2
Parts:
- removed U$1: (no value), BaseApp:5PIN_SOT23
- added C22, C23: 4.7u, rcl:C1206
- added IMU_3V3, IMU_3V3_, IMU_GND, IMU_GND_, IMU_INT1, IMU_SCL, IMU_SDA, SCL, SDA: TPTP10SQ, testpad:TP10SQ
- added MCP73831: (no value), BaseApp:5PIN_SOT23
- added R18: 2k, rcl:R0603
- added R19: 4k, rcl:R0603
- added R20, R21: 10k, rcl:R0603
- added STATUS: YL, led:CHIPLED_0603
- PWM1, PWM2, PWM3, PWM4: value TPTP10SQ -> TPTP12SQ; device testpad:TP10SQ -> testpad:TP12SQ
- REXT: value 135.45 -> 120
- moved PWM2 57.2 mm to (12.1, 29.5)
- moved PWM4 54.7 mm to (26.8, -9.94), turned to 45 degrees
- moved BAT+ 42.1 mm to (10.2, -21.0), turned to 90 degrees
- moved BAT- 38.3 mm to (7.30, -21.0), turned to 90 degrees
- moved PWM1 31.5 mm to (-17.8, 31.8)
- moved GND_PWM2 22.6 mm to (27.9, -11.7), turned to 225 degrees
- moved 3V3_PWM2 21.4 mm to (29.3, -13.7), turned to 45 degrees
- moved D3 19.7 mm to (-24.1, -22.2)
- moved T3 19.7 mm to (-21.0, -23.5)
- moved R13 19.7 mm to (-21.0, -20.3)
- moved TXD0 14.8 mm to (-10.2, -4.13)
- moved R2 14.2 mm to (0.32, -7.62), turned to 90 degrees
- moved PWR 13.5 mm to (0.32, -10.5), turned to 180 degrees
- moved INT1 13.4 mm to (-7.30, -5.08)
- moved 3V3 12.7 mm to (-1.27, -6.67), turned to 0 degrees
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Connections:
- removed net VBAT: BAT+.TP, CIN.2, D1.C, D2.C, D3.C, D4.C, M1+.TP, M2+.TP, M3+.TP, M4+.TP, R1.2, REXT.2, U1.1, U1.3
- new net BAT+: BAT+.TP, C23.2, MCP73831.P$3, R1.2
- new net N$2: MCP73831.P$1, STATUS.C
- new net N$3: R18.1, STATUS.A
- new net N$4: MCP73831.P$5, R19.1
- new net USBCNTRL: MC1.6, R20.1, R21.2
- net +3V3: now also IMU_3V3.TP, IMU_3V3_.TP
- net GND: now also C22.2, C23.1, IMU_GND.TP, IMU_GND_.TP, MCP73831.P$2, R19.2, R20.2
- net INT1: now also IMU_INT1.TP
- net PWM2: now also PWM4.TP; no longer PWM2.TP
- net PWM4: now also PWM2.TP; no longer PWM4.TP
- net SCL: now also IMU_SCL.TP, SCL.TP
- net SDA: now also IMU_SDA.TP, SDA.TP
- net V+: now also C22.1, MCP73831.P$4, R18.2, R21.1
- net VCC: now also CIN.2, D1.C, D2.C, D3.C, D4.C, M1+.TP, M2+.TP, M3+.TP, M4+.TP, REXT.2, U1.1, U1.3
Routing:
- net V+: track 0.00 -> 33.1 mm, vias 0 -> 2
- net PWM2: track 29.3 -> 0.00 mm, vias 2 -> 0
- net SCL: track 2.21 -> 29.5 mm, vias 0 -> 2
- net INT1: track 0.00 -> 26.0 mm
- net VBAT: track 25.0 -> 0.00 mm
- net SDA: track 2.40 -> 22.3 mm, vias 0 -> 4
- net USBCNTRL: track 0.00 -> 19.3 mm, vias 0 -> 2
- net BUSYLED3: track 41.0 -> 22.8 mm, vias 0 -> 2
- net AREF: track 19.7 -> 1.62 mm, vias 2 -> 0
- net BATCNTRL: track 18.1 -> 1.47 mm, vias 2 -> 0
- net PDI_CLOCK: track 14.0 -> 0.00 mm
- net +3V3: track 55.6 -> 69.1 mm, vias 0 -> 2
- net BUSYLED4: track 13.4 -> 0.00 mm
- net +5V: track 16.0 -> 5.62 mm
- net GND: track 77.1 -> 87.1 mm, vias 14 -> 19
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- added copper zone on layer 1, net VCC
- removed copper zone on layer 1, net VBAT
Other:
- outline, holes or cut-outs redrawn
- board text added: "EAZY EZBL-3A BL ESC"
