File: hardware/Schaltplan/Nanocopter_V2.sch (EAGLE design)
At the start: 86 parts, among them M1+ TPTP15SQ, M1- TPTP15SQ, M2+ TPTP15SQ, M2- TPTP15SQ, M3+ TPTP15SQ, M3- TPTP15SQ, M4+ TPTP15SQ, M4- TPTP15SQ, T1 IRLML2502, T2 IRLML2502, T3 IRLML2502, T4 IRLML2502, U1 MAX682, U2 PRTR5V0U2X, U3 LM3480-3.3, X1 USBSMD

Commit message: Arbeit an Schaltplan V2
Parts:
- removed U$1: (no value), BaseApp:MCP73831
- added C22, C23: 4.7u, rcl:C-EUC1206
- added IMU_3V3, IMU_3V3_, IMU_GND, IMU_GND_, IMU_INT1, IMU_SCL, IMU_SDA, SCL, SDA: TPTP10SQ, testpad:TPTP10SQ
- added MCP73831: (no value), BaseApp:MCP73831
- added R18: 2k, rcl:R-EU_R0603
- added R19: 4k, rcl:R-EU_R0603
- added R20, R21: 10k, rcl:R-EU_R0603
- added STATUS: YL, led:LEDCHIPLED_0603
- PWM1, PWM2, PWM3, PWM4: value TPTP10SQ -> TPTP12SQ; device testpad:TPTP10SQ -> testpad:TPTP12SQ
- REXT: value 135.45 -> 120
Connections:
- removed net VBAT: BAT+.TP, CIN.2, D1.C, D2.C, D3.C, D4.C, M1+.TP, M2+.TP, M3+.TP, M4+.TP, R1.2, REXT.2, U1.IN, U1.SKIP
- new net BAT+: BAT+.TP, C23.2, MCP73831.VBAT, R1.2
- new net N$2: MCP73831.STAT, STATUS.C
- new net N$3: R18.1, STATUS.A
- new net N$4: MCP73831.PROG, R19.1
- new net USBCNTRL: MC1.PB2(ADC10,DAC0), R20.1, R21.2
- net +3V3: now also IMU_3V3.TP, IMU_3V3_.TP
- net GND: now also C22.2, C23.1, IMU_GND.TP, IMU_GND_.TP, MCP73831.VSS, R19.2, R20.2
- net INT1: now also IMU_INT1.TP
- net PWM2: now also PWM4.TP; no longer PWM2.TP
- net PWM4: now also PWM2.TP; no longer PWM4.TP
- net SCL: now also IMU_SCL.TP, SCL.TP
- net SDA: now also IMU_SDA.TP, SDA.TP
- net V+: now also C22.1, MCP73831.VDD, R18.2, R21.1
- net VCC: now also CIN.2, D1.C, D2.C, D3.C, D4.C, M1+.TP, M2+.TP, M3+.TP, M4+.TP, REXT.2, U1.IN, U1.SKIP
Other:
- note added: "250mA Ladestrom"
- note added: "Beschleunigungs-, Gyrosensor und Kompass"
- note added: "LiPo USB Lader"
- note added: "Motoren unbedingt deaktivieren, wenn an USB angeschlossen -> ADC10!"
- note added: "Spannungskontroller und Referenz- spannung für ADC"
- note added: "Todo: Laderegler vom Rest der Schaltung trennen"
- note removed: "Beschleunigungs- und Gyrosensor"
- note removed: "Kontrolle der Batteriespannung"
- note removed: "USB Spannungsversorgung / Spannungsversorgung Batterie"
- note removed: "dies verhindert ein zu großer Stromverbrauch über USB"
- note removed: "erzeugt gleichzeitig die Referenzspannung für den ADC"
- moved on the sheet: BAT+, BAT-, D5, PWM2, PWM4, R1, R10, R9
