File: hardware/Schaltplan/Nanocopter_V2.1.brd (EAGLE design)
At the start: 100 x 100 mm, 87 parts, among them M1+ TPTP15SQ, M1- TPTP15SQ, M2+ TPTP15SQ, M2- TPTP15SQ, M3+ TPTP15SQ, M3- TPTP15SQ, M4+ TPTP15SQ, M4- TPTP15SQ, T1 IRLML2502, T2 IRLML2502, T3 IRLML2502, T4 IRLML2502, U2 PRTR5V0U2X, U3 LM3480-3.3, X1 USBSMD

Commit message: Neuer Schaltplan V2.1. Die Schaltung wird jetzt in zwei Teile aufgeteilt: Flugcontroller (SimpleControl) und Motortreiber-platine (BaseFrame).
Parts:
- removed BAT+, BAT-, GND_: TPTP12SQ, testpad:TP12SQ
- removed C22, C23: 4.7u, rcl:C1206
- removed D1, D2, D3, D4: (no value), diode:MINIMELF
- removed IMU_GND, IMU_INT1, IMU_SCL, IMU_SDA, INT1, RXD0, SCL, SDA, TXD0, XCK0: TPTP10SQ, testpad:TP10SQ
- removed LED1, LED2: BL, led:CHIPLED_0603
- removed LED3, LED4: RD, led:CHIPLED_0603
- removed M1+, M1-, M2+, M2-, M3+, M3-, M4+, M4-: TPTP15SQ, testpad:TP15SQ
- removed MCP73831: (no value), BaseApp:5PIN_SOT23
- removed PH1: PH1X6-05LONG, pel_hdr:PHL005-1-6
- removed R16, R17: 1k, rcl:R0603
- removed R18: 2k, rcl:R0603
- removed R19: 4k, rcl:R0603
- removed STATUS: YL, led:CHIPLED_0603
- removed T1, T2, T3, T4: IRLML2502, transistor-small-signal:SOT23
- added 3V1, 3V2, 3V4, 3V5, 3V6, 3V7, 3V8, GND_BASE2, PWM1, V+, V+_BASE: TPTP12SQ, testpad:TP12SQ
- added C4, C5: 10u, rcl:C1206
- added C6, C7: 10p, rcl:C0603
- added CRYSTAL1: (no value), BaseApp:CRYSTAL-4PIN
- added D6: BAT54C, diode:SOT23
- added JP10: (no value), pinhead:1X02
- added JP11: (no value), pinhead:1X02/90
- added JP14, JP15, JP16, JP17: (no value), pinhead:1X03/90
- added JP8, JP9: (no value), pinhead:1X03
- added L1+, L1-, L2+, L2-, L3+, L3-, L4+, L4-, M1A, M1B, M1C, M2A, M2B, M2C, M3A, M3B, M3C, M4A, M4B, M4C, VBAT+, VBAT-: TPSQTP20SQ, testpad:TP20SQ
- added LED5, LED6, STATUS2: RD, led:CHIPLED_0603
- added LED7, LED8: BL, led:CHIPLED_0603
- added MCP1: (no value), BaseApp:5PIN_SOT23
- added R22, R23, R24, R26: 10k, rcl:R0603
- added R27: 2k, rcl:R0603
- added R28: 4k, rcl:R0603
- added SJ2: (no value), jumper:SJ
- added SJ3: (no value), jumper:SJ_2
- added STATUS1: YL, led:CHIPLED_0603
- added T5, T6, T7, T8: IRLML2502, transistor-small-signal:SOT23
- added U$1, U$2, U$3, U$4: EAZY_BL_3A, eazy_bl_3A:EZ_BL_3A_P
- added U$5, U$6: IRF7321, irf:SO8
- added X2: 53261-08, con-molex:53261-08
- added X3, X6: 53261-06, con-molex:53261-06
- added X4, X5: 53261-03, con-molex:53261-03
- R11, R12: value 10k -> 2k
- R13, R14: value 10k -> 1k
- R3: value 2k -> 10k
- moved R15 201.8 mm to (89.9, -159.4), turned to 0 degrees
- moved R3 175.6 mm to (89.9, -154.6), turned to 0 degrees
- moved R11 131.5 mm to (43.8, -104.1)
- moved R14 127.7 mm to (39.1, -104.1), turned to 0 degrees
- moved GND 116.1 mm to (114.6, -18.4)
- moved R13 104.8 mm to (48.9, -98.4), turned to 0 degrees
- moved R12 99.0 mm to (44.1, -98.4), turned to 0 degrees
- moved MC1 70.8 mm to (-68.9, 4.13)
Connections:
- removed net +5V: PH1.6
- removed net PWM1_BASE: R11.1, T1.1
- removed net PWM2_BASE: R12.1, T2.1
- removed net PWM3_BASE: R13.1, T3.1
- removed net PWM4_BASE: R14.1, T4.1
- removed net RXD1: JP5.4, MC1.26, R8.2
- removed net TXD1: JP5.3, MC1.27, R7.2
- new net BUZZER: MC1.44, X3.6
- new net D+: JP5.3, MC1.27, R7.2, X5.3
- new net D-: JP5.4, MC1.26, R8.2, X5.2
- new net LED1: R22.1, T5.1, X6.5
- new net LED2: R23.1, T6.1, X6.4
- new net LED3: R24.1, T7.1, X6.3
- new net LED4: R26.1, T8.1, X6.2
- new net N$11: L1-.TP, LED8.C, T5.3
- new net N$12: L3-.TP, LED5.C, T7.3
- new net N$13: L4-.TP, LED6.C, T8.3
- new net N$14: L2-.TP, LED7.C, T6.3
- new net N$16: MCP1.P$5, R28.2
- new net N$20: C5.2, MCP1.P$3, SJ3.1, U$5.3, U$6.3
- new net N$23: R15.2, STATUS2.A
- new net N$24: M1A.TP, U$1.OUT_A
- new net N$25: M1B.TP, U$1.OUT_B
- new net N$26: M1C.TP, U$1.OUT_C
- new net N$27: JP15.3, U$2.IN_SIGNAL
- new net N$28: M3A.TP, U$3.OUT_A
- new net N$29: M3B.TP, U$3.OUT_B
- new net N$31: JP16.3, U$3.IN_SIGNAL
- new net N$32: M4A.TP, U$4.OUT_A
- new net N$33: M4B.TP, U$4.OUT_B
- new net N$34: M4C.TP, U$4.OUT_C
- new net N$35: JP17.3, U$4.IN_SIGNAL
- new net N$36: D6.1, SJ2.1
- new net N$37: R27.1, STATUS1.C
- new net N$38: MCP1.P$1, STATUS1.A, STATUS2.C
- new net N$39: SJ3.2, VBAT+.TP
- new net N$6: C3.1, D6.3, U3.2
- new net PD0: MC1.20, X2.2
- new net PD4: MC1.24, X2.7
- new net PD5: MC1.25, X2.8
- new net RXD2: MC1.32, X4.2
- new net TXD2: MC1.33, X4.3
- net BAT+: no longer BAT+.TP, C23.2, MCP73831.P$3
- net BUSYLED1: now also MC1.40, X3.2; no longer MC1.1, R17.2
- net BUSYLED2: now also MC1.41, X3.3; no longer R16.2
- net BUSYLED3: now also MC1.42, X3.4; no longer R3.2
- net BUSYLED4: now also MC1.43, X3.5; no longer R15.2
- net GND: now also C4.2, C5.1, C6.2, C7.2, GND_BASE2.TP, JP1.3, JP10.1, JP11.1, JP14.1, JP2.3, JP3.3, JP4.3, JP6.3, JP7.3, JP8.3, JP9.3, MCP1.P$2, R22.2, R23.2, R24.2, R26.2, R27.2, R28.1, R3.2, T5.2, T6.2, T7.2, T8.2, U$1.IN_M, U$2.IN_M, U$3.IN_M, U$4.IN_M, VBAT-.TP, X2.1, X3.1, X4.1, X5.1, X6.6; no longer BAT-.TP, C22.2, C23.1, GND_.TP, IMU_GND.TP, LED1.C, LED2.C, LED3.C, LED4.C, MCP73831.P$2, PH1.1, R11.2, R12.2, R13.2, R14.2, R19.2, T1.2, T2.2, T3.2, T4.2
- net INT1: now also MC1.3; no longer IMU_INT1.TP, INT1.TP, MC1.24
- net N$10: now also C7.1, CRYSTAL1.1, MC1.36; no longer LED3.A, R3.1
- net N$15: now also C6.1, CRYSTAL1.3, MC1.37; no longer LED4.A, R15.1
- net N$17: now also JP14.3, U$1.IN_SIGNAL; no longer LED2.A, R16.1
- net N$18: now also M2A.TP, U$2.OUT_A; no longer LED1.A, R17.1
- net N$19: now also LED8.A, R14.1; no longer D1.A, M1-.TP, T1.3
- net N$2: now also LED5.A, R11.1; no longer MCP73831.P$1, STATUS.C
- net N$21: now also M2B.TP, U$2.OUT_B; no longer D3.A, M3-.TP, T3.3
- net N$22: now also M2C.TP, U$2.OUT_C; no longer D4.A, M4-.TP, T4.3
- net N$3: now also LED6.A, R12.1; no longer R18.1, STATUS.A
- net N$30: now also M3C.TP, U$3.OUT_C; no longer D2.A, M2-.TP, T2.3
- net N$4: now also LED7.A, R13.1; no longer MCP73831.P$5, R19.1
- net PWM1: now also JP1.1, PWM1.TP
- net PWM2: now also 3V2.TP, JP2.1
- net PWM3: now also 3V4.TP, JP3.1
- net PWM4: now also 3V5.TP, JP4.1
- net PWM5: now also 3V1.TP, JP6.1
- net PWM6: now also 3V6.TP, JP7.1
- net PWM7: now also 3V7.TP, JP8.1
- net PWM8: now also 3V8.TP, JP9.1
- net RXD0: now also X2.4; no longer PH1.4, RXD0.TP
- net SCL: no longer IMU_SCL.TP, SCL.TP
- net SDA: no longer IMU_SDA.TP, SDA.TP
- net TXD0: now also X2.5; no longer TXD0.TP
- net V+: now also JP10.2, SJ2.2, V+.TP; no longer R18.2
- net VCC: now also D6.2, JP1.2, JP14.2, JP2.2, JP3.2, JP4.2, JP6.2, JP7.2, JP8.2, JP9.2, L1+.TP, L2+.TP, L3+.TP, L4+.TP, R11.2, R12.2, R13.2, R14.2, SJ3.3, U$1.IN_P, U$2.IN_P, U$3.IN_P, U$4.IN_P, U$5.5, U$5.6, U$5.7, U$5.8, U$6.5, U$6.6, U$6.7, U$6.8, X2.6; no longer C3.1, D1.C, D2.C, D3.C, D4.C, M1+.TP, M2+.TP, M3+.TP, M4+.TP, U3.2
- net VDD: now also C4.1, JP11.2, MCP1.P$4, R15.1, R3.1, U$5.1, U$5.2, U$5.4, U$6.1, U$6.2, U$6.4, V+_BASE.TP; no longer C22.1, MCP73831.P$4
- net XCK0: now also X2.3; no longer XCK0.TP
Routing:
- net GND: track 80.2 -> 30.5 mm, vias 18 -> 6
- net +3V3: track 65.5 -> 32.1 mm, vias 2 -> 0
- net BUSYLED3: track 21.6 -> 0.00 mm, vias 2 -> 0
- net RXD1: track 19.1 -> 0.00 mm, vias 1 -> 0
- net INT1: track 26.0 -> 7.29 mm
- net USBCNTRL: track 19.3 -> 1.59 mm, vias 2 -> 0
- net TXD1: track 15.8 -> 0.00 mm
- net SCL: track 29.5 -> 14.6 mm, vias 2 -> 0
- net SDA: track 22.3 -> 9.71 mm, vias 4 -> 2
- net BUSYLED2: track 12.2 -> 0.00 mm, vias 2 -> 0
- net RXD0: track 10.1 -> 0.00 mm
- net TXD0: track 8.29 -> 0.00 mm
- net XCK0: track 7.31 -> 0.00 mm
- net VDD: track 7.02 -> 0.00 mm
- net VCC: track 6.37 -> 0.00 mm
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- added copper zone on layer 1, net +3V3
Other:
- board size 100 x 100 mm -> 142 x 100 mm
- board text removed: "EAZY EZBL-3A BL ESC"
